Commit message: Collisions: base and art1

File: ws_thor/src/urdf_thor/urdf/thor.urdf (robot description, URDF)
Before this commit: robot THOR_arm, 7 links, 6 joints
Links:
- link art1: geometry collision box size=0.14 0.09 0.14; visual mesh filename=package://urdf_thor/meshes/art1.stl scale=0.001 0.001 0.001
- link base: geometry collision cylinder length=0.132 radius=0.096; visual mesh filename=package://urdf_thor/meshes/base.stl scale=0.001 0.001 0.001

Commit message: Art 2 collision mesh

File: ws_thor/src/urdf_thor/urdf/thor.urdf (robot description, URDF)
Before this commit: robot THOR_arm, 7 links, 6 joints
Links:
- link art2: geometry collision cylinder length=0.28 radius=0.085; visual mesh filename=package://urdf_thor/meshes/art2.stl scale=0.001 0.001 0.001

Commit message: Art4 collision mesh

File: ws_thor/src/urdf_thor/urdf/thor.urdf (robot description, URDF)
Before this commit: robot THOR_arm, 7 links, 6 joints
Links:
- link art4: geometry collision cylinder length=0.14 radius=0.065; visual mesh filename=package://urdf_thor/meshes/art4.stl scale=0.001 0.001 0.001

Commit message: Art6 collision mesh

File: ws_thor/src/urdf_thor/urdf/thor.urdf (robot description, URDF)
Before this commit: robot THOR_arm, 7 links, 6 joints
Links:
- link art6: geometry collision cylinder length=0.012 radius=0.025; visual mesh filename=package://urdf_thor/meshes/art6.stl scale=0.001 0.001 0.001
