Commit message: Hardware Controller added

File: ws_thor/src/moveit_thor/config/THOR_arm.ros2_control.xacro (robot description, xacro)
@@ -1,60 +1,54 @@
 <?xml version="1.0"?>
-<robot xmlns:xacro="http://www.ros.org/wiki/xacro">
-    <xacro:macro name="THOR_arm_ros2_control" params="name initial_positions_file">
-        <xacro:property name="initial_positions" value="${load_yaml(initial_positions_file)['initial_positions']}"/>
-        <ros2_control name="${name}" type="system">
-            <hardware>
-                <!-- By default, set up controllers for simulation. This won't work on real hardware -->
-                <plugin>mock_components/GenericSystem</plugin>
-            </hardware>
-            <joint name="art1_yaw">
-                <command_interface name="position"/>
-                <command_interface name="velocity"/>
-                <state_interface name="position">
-                  <param name="initial_value">${initial_positions['art1_yaw']}</param>
-                </state_interface>
-                <state_interface name="velocity"/>
-            </joint>
-            <joint name="art2_pitch">
-                <command_interface name="position"/>
-                <command_interface name="velocity"/>
-                <state_interface name="position">
-                  <param name="initial_value">${initial_positions['art2_pitch']}</param>
-                </state_interface>
-                <state_interface name="velocity"/>
-            </joint>
-            <joint name="art3_pitch">
-                <command_interface name="position"/>
-                <command_interface name="velocity"/>
-                <state_interface name="position">
-                  <param name="initial_value">${initial_positions['art3_pitch']}</param>
-                </state_interface>
-                <state_interface name="velocity"/>
-            </joint>
-            <joint name="art4_roll">
-                <command_interface name="position"/>
-                <command_interface name="velocity"/>
-                <state_interface name="position">
-                  <param name="initial_value">${initial_positions['art4_roll']}</param>
-                </state_interface>
-                <state_interface name="velocity"/>
-            </joint>
-            <joint name="art5_pitch">
-                <command_interface name="position"/>
-                <command_interface name="velocity"/>
-                <state_interface name="position">
-                  <param name="initial_value">${initial_positions['art5_pitch']}</param>
-                </state_interface>
-                <state_interface name="velocity"/>
-            </joint>
-            <joint name="art6_roll">
-                <command_interface name="position"/>
-                <command_interface name="velocity"/>
-                <state_interface name="position">
-                  <param name="initial_value">${initial_positions['art6_roll']}</param>
-                </state_interface>
-                <state_interface name="velocity"/>
-            </joint>
-        </ros2_control>
-    </xacro:macro>
+<robot xmlns:xacro="http://www.ros.org/wiki/xacro" name="THOR_arm">
+  <ros2_control name="RobotSystem" type="system">
+    <!-- HARDWARE -->
+    <xacro:if value="$(arg is_sim)">
+        <hardware>
+            <plugin>gazebo_ros2_control/GazeboSystem</plugin>
+        </hardware>
+    </xacro:if>
+    <xacro:unless value="$(arg is_sim)">
+        <hardware>
+            <plugin>thor_controller/ThorInterface</plugin>
+            <param name="port">/dev/ttyACM0</param>
+        </hardware>
+    </xacro:unless>
+    <!-- JOINTS -->
+    <joint name="art1_yaw">
+        <command_interface name="position"/>
+        <!--<command_interface name="velocity"/>-->
+        <state_interface name="position"/>
+        <!--<state_interface name="velocity"/>-->
+    </joint>
+    <joint name="art2_pitch">
+        <command_interface name="position"/>
+        <!--<command_interface name="velocity"/>-->
+        <state_interface name="position"/>
+        <!--<state_interface name="velocity"/>-->
+    </joint>
+    <joint name="art3_pitch">
+        <command_interface name="position"/>
+        <!--<command_interface name="velocity"/>-->
+        <state_interface name="position"/>
+        <!--<state_interface name="velocity"/>-->
+    </joint>
+    <joint name="art4_roll">
+        <command_interface name="position"/>
+        <!--<command_interface name="velocity"/>-->
+        <state_interface name="position"/>
+        <!--<state_interface name="velocity"/>-->
+    </joint>
+    <joint name="art5_pitch">
+        <command_interface name="position"/>
+        <!--<command_interface name="velocity"/>-->
+        <state_interface name="position"/>
+        <!--<state_interface name="velocity"/>-->
+    </joint>
+    <joint name="art6_roll">
+        <command_interface name="position"/>
+        <!--<command_interface name="velocity"/>-->
+        <state_interface name="position"/>
+        <!--<state_interface name="velocity"/>-->
+    </joint>
+  </ros2_control>
 </robot>

File: ws_thor/src/urdf_thor/urdf/thor.urdf.xacro (robot description, xacro)
@@ -1,6 +1,34 @@
 <?xml version="1.0"?>
-<robot name="THOR_arm">
+<robot xmlns:xacro="http://www.ros.org/wiki/xacro" name="THOR_arm">
+  <!-- Load Simulated or Real Hardware Interfaces -->
+  <xacro:arg name="is_sim" default="true"/>
+  <!-- Include Gazebo Parameters -->
+  <xacro:include filename="$(find urdf_thor)/urdf/thor_gazebo.xacro" />
+  <!-- Include ros2_control Plugins -->
+  <xacro:include filename="$(find moveit_thor)/config/THOR_arm.ros2_control.xacro" />
+  <!-- Useful XACRO Variables (Properties) -->
+  <xacro:property name="PI" value="3.14159265359" />
+  <xacro:property name="effort" value="30.0" />
+  <xacro:property name="velocity" value="10.0" />
+  <!-- Useful Macros -->
+  <xacro:macro name="default_inertial" params="mass">
+      <inertial>
+          <origin xyz="0 0 0" rpy="0 0 0"/>
+          <mass value="${mass}" />
+          <inertia ixx="1.0" ixy="0.0" ixz="0.0"
+                  iyy="1.0" iyz="0.0"
+                  izz="1.0" />
+      </inertial>
+  </xacro:macro>
+  <!-- World Link -->
+  <link name="world"/>
+  <joint name="virtual_joint" type="fixed">
+    <parent link="world"/>
+    <child link="base"/>
+    <origin xyz="0 0 0" rpy="0 0 0"/>
+  </joint>
   <!-- Link robot base -->
   <link name="base">
+    <xacro:default_inertial mass="1.0"/>
     <visual>
       <origin xyz="0 0 0" rpy="0 0 0"/>
@@ -29,4 +57,5 @@
   <!-- Link art1 -->
   <link name="art1">
+    <xacro:default_inertial mass="1.0"/>
     <visual>
       <origin xyz="0 0 0" rpy="0 0 0" />
@@ -53,4 +82,5 @@
   <!-- Link art2 -->
   <link name="art2">
+    <xacro:default_inertial mass="1.0"/>
     <visual>
       <origin xyz="0 0 0" rpy="0 0 0" />
@@ -77,4 +107,5 @@
   <!-- Link art3 -->
   <link name="art3">
+    <xacro:default_inertial mass="1.0"/>
     <visual>
       <origin xyz="0 0 0" rpy="0 0 0" />
@@ -95,4 +126,5 @@
   <!-- Link art4 -->
   <link name="art4">
+    <xacro:default_inertial mass="1.0"/>
     <visual>
       <origin xyz="0 0 0" rpy="0 0 0" />
@@ -119,4 +151,5 @@
   <!-- Link art5 -->
   <link name="art5">
+    <xacro:default_inertial mass="1.0"/>
     <visual>
       <origin xyz="0 0 0" rpy="0 0 0" />
@@ -137,4 +170,5 @@
   <!-- Link art6 -->
   <link name="art6">
+    <xacro:default_inertial mass="1.0"/>
     <visual>
       <origin xyz="0 0 0" rpy="0 0 0" />
