Commit message: renamed urdf_thor to thor_urdf to maintain consistency with the rest of the packages.

File: ws_thor/src/moveit_thor/config/THOR_arm.urdf.xacro (robot description, xacro)
@@ -3,5 +3,5 @@
     <xacro:arg name="initial_positions_file" default="initial_positions.yaml" />
     <!-- Import THOR_arm urdf file -->
-    <xacro:include filename="$(find urdf_thor)/urdf/thor.urdf" />
+    <xacro:include filename="$(find thor_urdf)/urdf/thor.urdf" />
     <!-- Import control_xacro -->
     <xacro:include filename="THOR_arm.ros2_control.xacro" />

File: ws_thor/src/thor_urdf/urdf/thor.urdf.xacro (robot description, xacro)
@@ -4,5 +4,5 @@
   <xacro:arg name="is_sim" default="true"/>
   <!-- Include Gazebo Parameters -->
-  <xacro:include filename="$(find urdf_thor)/urdf/thor_gazebo.xacro" />
+  <xacro:include filename="$(find thor_urdf)/urdf/thor_gazebo.xacro" />
   <!-- Include ros2_control Plugins -->
   <xacro:include filename="$(find moveit_thor)/config/THOR_arm.ros2_control.xacro" />
@@ -34,5 +34,5 @@
       <origin xyz="0 0 0" rpy="0 0 -${PI / 2}"/>
       <geometry>
-        <mesh filename="package://urdf_thor/meshes/Base.dae" scale="0.001 0.001 0.001" />
+        <mesh filename="package://thor_urdf/meshes/Base.dae" scale="0.001 0.001 0.001" />
       </geometry>
     </visual>
@@ -64,5 +64,5 @@
       <origin xyz="0 0 0" rpy="0 0 -${PI / 2}"/>
       <geometry>
-        <mesh filename="package://urdf_thor/meshes/Art1.dae" scale="0.001 0.001 0.001" />
+        <mesh filename="package://thor_urdf/meshes/Art1.dae" scale="0.001 0.001 0.001" />
       </geometry>
     </visual>
@@ -88,5 +88,5 @@
       <origin xyz="0 0 0" rpy="0 0 -${PI / 2}"/>
       <geometry>
-        <mesh filename="package://urdf_thor/meshes/Art2.dae" scale="0.001 0.001 0.001" />
+        <mesh filename="package://thor_urdf/meshes/Art2.dae" scale="0.001 0.001 0.001" />
       </geometry>
     </visual>
@@ -124,5 +124,5 @@
       <origin xyz="0 0 0" rpy="0 0 -${PI / 2}"/>
       <geometry>
-        <mesh filename="package://urdf_thor/meshes/Art3.dae" scale="0.001 0.001 0.001" />
+        <mesh filename="package://thor_urdf/meshes/Art3.dae" scale="0.001 0.001 0.001" />
       </geometry>
     </visual>
@@ -148,5 +148,5 @@
       <origin xyz="0 0 0" rpy="0 0 -${PI / 2}"/>
       <geometry>
-        <mesh filename="package://urdf_thor/meshes/Art4.dae" scale="0.001 0.001 0.001" />
+        <mesh filename="package://thor_urdf/meshes/Art4.dae" scale="0.001 0.001 0.001" />
       </geometry>
     </visual>
@@ -184,5 +184,5 @@
       <origin xyz="0 0 0" rpy="0 0 -${PI / 2}"/>
       <geometry>
-          <mesh filename="package://urdf_thor/meshes/Art5.dae" scale="0.001 0.001 0.001" />
+          <mesh filename="package://thor_urdf/meshes/Art5.dae" scale="0.001 0.001 0.001" />
       </geometry>
     </visual>
@@ -208,5 +208,5 @@
       <origin xyz="0 0 0" rpy="0 0 -${PI / 2}"/>
       <geometry>
-          <mesh filename="package://urdf_thor/meshes/Art6.dae" scale="0.001 0.001 0.001" />
+          <mesh filename="package://thor_urdf/meshes/Art6.dae" scale="0.001 0.001 0.001" />
       </geometry>
     </visual>
