Commit message: Gripper added

File: ws_thor/src/thor_moveit/config/THOR_arm.ros2_control.xacro (robot description, xacro)
@@ -7,4 +7,24 @@
             <plugin>gazebo_ros2_control/GazeboSystem</plugin>
         </hardware>
+        <joint name="gripperbase_to_armgearleft">
+                <param name="mimic">gripperbase_to_armgearright</param>
+                <param name="multiplier">-1</param>
+        </joint>
+        <joint name="gripperbase_to_armsimpleright">
+                <param name="mimic">gripperbase_to_armgearright</param>
+                <param name="multiplier">1</param>
+        </joint>
+        <joint name="gripperbase_to_armsimpleleft">
+                <param name="mimic">gripperbase_to_armgearright</param>
+                <param name="multiplier">-1</param>
+        </joint>
+        <joint name="armgearright_to_fingerright">
+                <param name="mimic">gripperbase_to_armgearright</param>
+                <param name="multiplier">-1</param>
+        </joint>
+        <joint name="armgearleft_to_fingerleft">
+                <param name="mimic">gripperbase_to_armgearright</param>
+                <param name="multiplier">-1</param>
+        </joint>
     </xacro:if>
     <xacro:unless value="$(arg is_sim)">
@@ -15,5 +35,5 @@
     </xacro:unless>
     <!-- JOINTS -->
-    <joint name="art1_yaw">
+    <joint name="joint_1">
         <command_interface name="position"/>
         <!--<command_interface name="velocity"/>-->
@@ -21,5 +41,5 @@
         <!--<state_interface name="velocity"/>-->
     </joint>
-    <joint name="art2_pitch">
+    <joint name="joint_2">
         <command_interface name="position"/>
         <!--<command_interface name="velocity"/>-->
@@ -27,5 +47,5 @@
         <!--<state_interface name="velocity"/>-->
     </joint>
-    <joint name="art3_pitch">
+    <joint name="joint_3">
         <command_interface name="position"/>
         <!--<command_interface name="velocity"/>-->
@@ -33,5 +53,5 @@
         <!--<state_interface name="velocity"/>-->
     </joint>
-    <joint name="art4_roll">
+    <joint name="joint_4">
         <command_interface name="position"/>
         <!--<command_interface name="velocity"/>-->
@@ -39,5 +59,5 @@
         <!--<state_interface name="velocity"/>-->
     </joint>
-    <joint name="art5_pitch">
+    <joint name="joint_5">
         <command_interface name="position"/>
         <!--<command_interface name="velocity"/>-->
@@ -45,5 +65,11 @@
         <!--<state_interface name="velocity"/>-->
     </joint>
-    <joint name="art6_roll">
+    <joint name="joint_6">
+        <command_interface name="position"/>
+        <!--<command_interface name="velocity"/>-->
+        <state_interface name="position"/>
+        <!--<state_interface name="velocity"/>-->
+    </joint>
+    <joint name="gripperbase_to_armgearright">
         <command_interface name="position"/>
         <!--<command_interface name="velocity"/>-->

File: ws_thor/src/thor_urdf/urdf/thor.urdf.xacro (robot description, xacro)
@@ -1,220 +1,391 @@
 <?xml version="1.0"?>
 <robot xmlns:xacro="http://www.ros.org/wiki/xacro" name="THOR_arm">
-  <!-- Load Simulated or Real Hardware Interfaces -->
-  <xacro:arg name="is_sim" default="true"/>
-  <!-- Include Gazebo Parameters -->
-  <xacro:include filename="$(find thor_urdf)/urdf/thor_gazebo.xacro" />
-  <!-- Include ros2_control Plugins -->
-  <xacro:include filename="$(find thor_moveit)/config/THOR_arm.ros2_control.xacro" />
-  <!-- Useful XACRO Variables (Properties) -->
-  <xacro:property name="PI" value="3.14159265359" />
-  <xacro:property name="effort" value="4.0" />
-  <xacro:property name="velocity" value="1.0" />
-  <!-- Useful Macros -->
-  <xacro:macro name="default_inertial" params="mass">
-      <inertial>
-          <origin xyz="0 0 0" rpy="0 0 0"/>
-          <mass value="${mass}" />
-          <inertia ixx="1.0" ixy="0.0" ixz="0.0"
-                  iyy="1.0" iyz="0.0"
-                  izz="1.0" />
-      </inertial>
-  </xacro:macro>
-  <!-- World Link -->
-  <link name="world"/>
-  <joint name="virtual_joint" type="fixed">
-    <parent link="world"/>
-    <child link="base"/>
-    <origin xyz="0 0 0" rpy="0 0 0"/>
-  </joint>
-  <!-- Link robot base -->
-  <link name="base">
-    <xacro:default_inertial mass="1.0"/>
-    <visual>
-      <origin xyz="0 0 0" rpy="0 0 -${PI / 2}"/>
-      <geometry>
-        <mesh filename="package://thor_urdf/meshes/Base.dae" scale="0.001 0.001 0.001" />
-      </geometry>
-    </visual>
-    <collision>
-        <origin xyz="0 0 0.049" rpy="0 0 -${PI / 2}"/>
-        <geometry>
-            <cylinder radius="0.075" length="0.098"/>
-        </geometry>
-    </collision>
-    <collision>
-        <origin xyz="0 -0.1312686 0.035250" rpy="0 0 -${PI / 2}"/>
-        <geometry>
-            <box size="0.176 0.180 0.0705"/>
-        </geometry>
-    </collision>
-  </link>
-  <!-- Joint base_art1 -->
-  <joint name="art1_yaw" type="revolute">
-    <origin xyz="0 0 0.099" rpy="0 0 0"/>
-    <axis xyz="0 0 1"/>
-    <parent link="base"/>
-    <child link="art1"/>
-    <limit lower="-2.967" upper="2.967" effort="${effort}" velocity="${velocity}"/>
-  </joint>
-  <!-- Link art1 -->
-  <link name="art1">
-    <xacro:default_inertial mass="1.0"/>
-    <visual>
-      <origin xyz="0 0 0" rpy="0 0 -${PI / 2}"/>
-      <geometry>
-        <mesh filename="package://thor_urdf/meshes/Art1.dae" scale="0.001 0.001 0.001" />
-      </geometry>
-    </visual>
-    <collision>
-        <origin xyz="0 0 0.0765" rpy="0 0 -${PI / 2}"/>
-        <geometry>
-            <cylinder radius="0.075" length="0.179"/>
-        </geometry>
-    </collision>
-  </link>
-  <!-- Joint art1_art2 -->
-  <joint name="art2_pitch" type="revolute">
-    <origin xyz="0 0 0.103" rpy="0 0 0"/>
-    <axis xyz="1 0 0"/>
-    <parent link="art1"/>
-    <child link="art2"/>
-    <limit lower="-${PI / 2}" upper="${PI / 2}" effort="${effort}" velocity="${velocity}"/>
-  </joint>
-  <!-- Link art2 -->
-  <link name="art2">
-    <xacro:default_inertial mass="1.0"/>
-    <visual>
-      <origin xyz="0 0 0" rpy="0 0 -${PI / 2}"/>
-      <geometry>
-        <mesh filename="package://thor_urdf/meshes/Art2.dae" scale="0.001 0.001 0.001" />
-      </geometry>
-    </visual>
-    <collision>
-        <origin xyz="0 0 0" rpy="${PI / 2} 0 -${PI / 2}"/>
-        <geometry>
-            <cylinder radius="0.065" length="0.140"/>
-        </geometry>
-    </collision>
-    <collision>
-        <origin xyz="0 0 0.080" rpy="${PI / 2} 0 -${PI / 2}"/>
-        <geometry>
-            <box size="0.130 0.160 0.140"/>
-        </geometry>
-    </collision>
-    <collision>
-        <origin xyz="0 0 0.160" rpy="${PI / 2} 0 -${PI / 2}"/>
-        <geometry>
-            <cylinder radius="0.065" length="0.140"/>
-        </geometry>
-    </collision>
-  </link>
-  <!-- Joint art2_art3 -->
-  <joint name="art3_pitch" type="revolute">
-    <origin xyz="0 0 0.160" rpy="0 0 0"/>
-    <axis xyz="1 0 0"/>
-    <parent link="art2"/>
-    <child link="art3"/>
-    <limit lower="-${PI / 2}" upper="${PI / 2}" effort="${effort}" velocity="${velocity}"/>
-  </joint>
-  <!-- Link art3 -->
-  <link name="art3">
-    <xacro:default_inertial mass="1.0"/>
-    <visual>
-      <origin xyz="0 0 0" rpy="0 0 -${PI / 2}"/>
-      <geometry>
-        <mesh filename="package://thor_urdf/meshes/Art3.dae" scale="0.001 0.001 0.001" />
-      </geometry>
-    </visual>
-    <collision>
-        <origin xyz="0 0 0.01225" rpy="0 0 -${PI / 2}"/>
-        <geometry>
-            <cylinder radius="0.055" length="0.1525"/>
-        </geometry>
-    </collision>
-  </link>
-  <!-- Joint art3_art4 -->
-  <joint name="art4_roll" type="revolute">
-    <origin xyz="0 0 0.0895" rpy="0 0 0"/>
-    <axis xyz="0 0 1"/>
-    <parent link="art3"/>
-    <child link="art4"/>
-    <limit lower="-2.967" upper="2.967" effort="${effort}" velocity="${velocity}"/>
-  </joint>
-  <!-- Link art4 -->
-  <link name="art4">
-    <xacro:default_inertial mass="1.0"/>
-    <visual>
-      <origin xyz="0 0 0" rpy="0 0 -${PI / 2}"/>
-      <geometry>
-        <mesh filename="package://thor_urdf/meshes/Art4.dae" scale="0.001 0.001 0.001" />
-      </geometry>
-    </visual>
-    <collision>
-        <origin xyz="0 0 0.1045" rpy="0 0 -${PI / 2}"/>
-        <geometry>
-            <sphere radius="0.055"/>
-        </geometry>
-    </collision>
-    <collision>
-        <origin xyz="0 0 0.05525" rpy="0 0 -${PI / 2}"/>
-        <geometry>
-            <cylinder radius="0.055" length="0.1045"/>
-        </geometry>
-    </collision>
-    <collision>
-        <origin xyz="0 0 0.0295" rpy="0 0 -${PI / 2}"/>
-        <geometry>
-            <box size="0.050 0.132 0.050"/>
-        </geometry>
-    </collision>
-  </link>
-  <!-- Joint art4_art5 -->
-  <joint name="art5_pitch" type="revolute">
-    <origin xyz="0 0 0.1045" rpy="0 0 0"/>
-    <axis xyz="1 0 0"/>
-    <parent link="art4"/>
-    <child link="art5"/>
-    <limit lower="-${PI / 2}" upper="${PI / 2}" effort="${effort}" velocity="${velocity}"/>
-  </joint>
-  <!-- Link art5 -->
-  <link name="art5">
-    <xacro:default_inertial mass="1.0"/>
-    <visual>
-      <origin xyz="0 0 0" rpy="0 0 -${PI / 2}"/>
-      <geometry>
-          <mesh filename="package://thor_urdf/meshes/Art5.dae" scale="0.001 0.001 0.001" />
-      </geometry>
-    </visual>
-    <collision>
-        <origin xyz="0 0 0" rpy="${PI / 2} 0 -${PI / 2}"/>
-        <geometry>
-            <cylinder radius="0.047" length="0.03"/>
-        </geometry>
-    </collision>
-  </link>
-  <!-- Joint art5_art6 -->
-  <joint name="art6_roll" type="revolute">
-    <origin xyz="0 0 0.0135" rpy="0 0 0"/>
-    <axis xyz="0 0 1"/>
-    <parent link="art5"/>
-    <child link="art6"/>
-    <limit lower="-2.967" upper="2.967" effort="${effort}" velocity="${velocity}"/>
-  </joint>
-  <!-- Link art6 -->
-  <link name="art6">
-    <xacro:default_inertial mass="1.0"/>
-    <visual>
-      <origin xyz="0 0 0" rpy="0 0 -${PI / 2}"/>
-      <geometry>
-          <mesh filename="package://thor_urdf/meshes/Art6.dae" scale="0.001 0.001 0.001" />
-      </geometry>
-    </visual>
-    <collision>
-        <origin xyz="0 0 0.025" rpy="0 0 -${PI / 2}"/>
-        <geometry>
-            <cylinder radius="0.015" length="0.05"/>
-        </geometry>
-    </collision>
-  </link>
+    <!-- Load Simulated or Real Hardware Interfaces -->
+    <xacro:arg name="is_sim" default="true"/>
+    <!-- Include Gazebo Parameters -->
+    <xacro:include filename="$(find thor_urdf)/urdf/thor_gazebo.xacro" />
+    <!-- Include ros2_control Plugins -->
+    <xacro:include filename="$(find thor_moveit)/config/THOR_arm.ros2_control.xacro" />
+    <!-- Useful XACRO Variables (Properties) -->
+    <xacro:property name="PI" value="3.14159265359" />
+    <xacro:property name="effort" value="4.0" />
+    <xacro:property name="velocity" value="1.0" />
+    <!-- Useful Macros -->
+    <xacro:macro name="default_inertial" params="mass">
+        <inertial>
+            <origin xyz="0 0 0" rpy="0 0 0"/>
+            <mass value="${mass}" />
+            <inertia ixx="1.0" ixy="0.0" ixz="0.0"
+                     iyy="1.0" iyz="0.0"
+                     izz="1.0" />
+        </inertial>
+    </xacro:macro>
+    <!-- Links -->
+    <link name="world"/>
+    <link name="base_link">
+        <xacro:default_inertial mass="1.0"/>
+        <visual>
+            <origin xyz="0 0 0" rpy="0 0 -${PI / 2}"/>
+            <geometry>
+              <mesh filename="package://thor_urdf/meshes/Base.dae" scale="0.001 0.001 0.001" />
+            </geometry>
+        </visual>
+        <collision>
+            <origin xyz="0 0 0.049" rpy="0 0 -${PI / 2}"/>
+            <geometry>
+                <cylinder radius="0.075" length="0.098"/>
+            </geometry>
+        </collision>
+        <collision>
+            <origin xyz="0 -0.1312686 0.035250" rpy="0 0 -${PI / 2}"/>
+            <geometry>
+                <box size="0.176 0.180 0.0705"/>
+            </geometry>
+        </collision>
+    </link>
+    <link name="link_1">
+        <xacro:default_inertial mass="1.0"/>
+        <visual>
+            <origin xyz="0 0 0" rpy="0 0 -${PI / 2}"/>
+            <geometry>
+              <mesh filename="package://thor_urdf/meshes/Art1.dae" scale="0.001 0.001 0.001" />
+            </geometry>
+        </visual>
+        <collision>
+            <origin xyz="0 0 0.0765" rpy="0 0 -${PI / 2}"/>
+            <geometry>
+                <cylinder radius="0.075" length="0.179"/>
+            </geometry>
+        </collision>
+    </link>
+    <link name="link_2">
+        <xacro:default_inertial mass="1.0"/>
+        <visual>
+            <origin xyz="0 0 0" rpy="0 0 -${PI / 2}"/>
+            <geometry>
+              <mesh filename="package://thor_urdf/meshes/Art2.dae" scale="0.001 0.001 0.001" />
+            </geometry>
+        </visual>
+        <collision>
+            <origin xyz="0 0 0" rpy="${PI / 2} 0 -${PI / 2}"/>
+            <geometry>
+                <cylinder radius="0.065" length="0.140"/>
+            </geometry>
+        </collision>
+        <collision>
+            <origin xyz="0 0 0.080" rpy="${PI / 2} 0 -${PI / 2}"/>
+            <geometry>
+                <box size="0.130 0.160 0.140"/>
+            </geometry>
+        </collision>
+        <collision>
+            <origin xyz="0 0 0.160" rpy="${PI / 2} 0 -${PI / 2}"/>
+            <geometry>
+                <cylinder radius="0.065" length="0.140"/>
+            </geometry>
+        </collision>
+    </link>
+    <link name="link_3">
+        <xacro:default_inertial mass="1.0"/>
+        <visual>
+            <origin xyz="0 0 0" rpy="0 0 -${PI / 2}"/>
+            <geometry>
+              <mesh filename="package://thor_urdf/meshes/Art3.dae" scale="0.001 0.001 0.001" />
+            </geometry>
+        </visual>
+        <collision>
+            <origin xyz="0 0 0.01225" rpy="0 0 -${PI / 2}"/>
+            <geometry>
+                <cylinder radius="0.055" length="0.1525"/>
+            </geometry>
+        </collision>
+    </link>
+    <link name="link_4">
+        <xacro:default_inertial mass="1.0"/>
+        <visual>
+            <origin xyz="0 0 0" rpy="0 0 -${PI / 2}"/>
+            <geometry>
+              <mesh filename="package://thor_urdf/meshes/Art4.dae" scale="0.001 0.001 0.001" />
+            </geometry>
+        </visual>
+        <collision>
+            <origin xyz="0 0 0.1045" rpy="0 0 -${PI / 2}"/>
+            <geometry>
+                <sphere radius="0.055"/>
+            </geometry>
+        </collision>
+        <collision>
+            <origin xyz="0 0 0.05525" rpy="0 0 -${PI / 2}"/>
+            <geometry>
+                <cylinder radius="0.055" length="0.1045"/>
+            </geometry>
+        </collision>
+        <collision>
+            <origin xyz="0 0 0.0295" rpy="0 0 -${PI / 2}"/>
+            <geometry>
+                <box size="0.050 0.132 0.050"/>
+            </geometry>
+        </collision>
+    </link>
+    <link name="link_5">
+        <xacro:default_inertial mass="1.0"/>
+        <visual>
+            <origin xyz="0 0 0" rpy="0 0 -${PI / 2}"/>
+            <geometry>
+                <mesh filename="package://thor_urdf/meshes/Art5.dae" scale="0.001 0.001 0.001" />
+            </geometry>
+        </visual>
+        <collision>
+            <origin xyz="0 0 0" rpy="${PI / 2} 0 -${PI / 2}"/>
+            <geometry>
+                <cylinder radius="0.047" length="0.03"/>
+            </geometry>
+        </collision>
+    </link>
+    <link name="link_6">
+        <xacro:default_inertial mass="1.0"/>
+        <visual>
+            <origin xyz="0 0 0" rpy="0 0 -${PI / 2}"/>
+        <geometry>
+            <mesh filename="package://thor_urdf/meshes/Art6.dae" scale="0.001 0.001 0.001" />
+        </geometry>
+        </visual>
+        <collision>
+            <origin xyz="0 0 0.025" rpy="0 0 -${PI / 2}"/>
+            <geometry>
+                <cylinder radius="0.015" length="0.05"/>
+            </geometry>
+        </collision>
+    </link>
+    <link name="gripper_base">
+        <xacro:default_inertial mass="1.0"/>
+        <visual>
+            <origin xyz="0 0 0" rpy="0 0 0"/>
+        <geometry>
+            <mesh filename="package://thor_urdf/meshes/GripperBase.dae" scale="0.001 0.001 0.001" />
+        </geometry>
+        </visual>
+        <!--
+        <collision>
+            <origin xyz="0 0 0.025" rpy="0 0 -${PI / 2}"/>
+            <geometry>
+                <cylinder radius="0.015" length="0.05"/>
+            </geometry>
+        </collision>
+        -->
+    </link>
+    <link name="gripper_arm_gear_right">
+        <xacro:default_inertial mass="1.0"/>
+        <visual>
+            <origin xyz="0 0 0" rpy="0 -${PI / 2} ${PI / 2}"/>
+        <geometry>
+            <mesh filename="package://thor_urdf/meshes/GripperArmGear.dae" scale="0.001 0.001 0.001" />
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