Commit message: Colliders for gripper parts added

File: ws_thor/src/thor_urdf/urdf/thor.urdf.xacro (robot description, xacro)
@@ -166,12 +166,16 @@
         </geometry>
         </visual>
-        <!--
-        <collision>
-            <origin xyz="0 0 0.025" rpy="0 0 -${PI / 2}"/>
-            <geometry>
-                <cylinder radius="0.015" length="0.05"/>
-            </geometry>
-        </collision>
-        -->
+        <collision>
+            <origin xyz="0 0 0.0275" rpy="0 0 0"/>
+            <geometry>
+                <box size="0.065 0.0348 0.055"/>
+            </geometry>
+        </collision>
+        <collision>
+            <origin xyz="-0.004250 0.03125 0.0325" rpy="0 0 0"/>
+            <geometry>
+                <box size="0.0406 0.0277 0.020"/>
+            </geometry>
+        </collision>
     </link>
     <link name="gripper_arm_gear_right">
@@ -183,12 +187,10 @@
         </geometry>
         </visual>
-        <!--
-        <collision>
-            <origin xyz="0 0 0.025" rpy="0 0 -${PI / 2}"/>
-            <geometry>
-                <cylinder radius="0.015" length="0.05"/>
-            </geometry>
-        </collision>
-        -->
+        <collision>
+            <origin xyz="0.0175 -0.0025 0.0" rpy="0 0 0"/>
+            <geometry>
+                <box size="0.035 0.005 0.004"/>
+            </geometry>
+        </collision>
     </link>
     <link name="gripper_arm_gear_left">
@@ -200,12 +202,10 @@
         </geometry>
         </visual>
-        <!--
-        <collision>
-            <origin xyz="0 0 0.025" rpy="0 0 -${PI / 2}"/>
-            <geometry>
-                <cylinder radius="0.015" length="0.05"/>
-            </geometry>
-        </collision>
-        -->
+        <collision>
+            <origin xyz="-0.0175 -0.0025 0.0" rpy="0 0 0"/>
+            <geometry>
+                <box size="0.035 0.005 0.004"/>
+            </geometry>
+        </collision>
     </link>
     <link name="gripper_arm_simple_right">
@@ -217,12 +217,10 @@
         </geometry>
         </visual>
-        <!--
-        <collision>
-            <origin xyz="0 0 0.025" rpy="0 0 -${PI / 2}"/>
-            <geometry>
-                <cylinder radius="0.015" length="0.05"/>
-            </geometry>
-        </collision>
-        -->
+        <collision>
+            <origin xyz="0.0175 -0.0025 0.0" rpy="0 0 0"/>
+            <geometry>
+                <box size="0.035 0.005 0.004"/>
+            </geometry>
+        </collision>
     </link>
     <link name="gripper_arm_simple_left">
@@ -234,12 +232,10 @@
         </geometry>
         </visual>
-        <!--
-        <collision>
-            <origin xyz="0 0 0.025" rpy="0 0 -${PI / 2}"/>
-            <geometry>
-                <cylinder radius="0.015" length="0.05"/>
-            </geometry>
-        </collision>
-        -->
+        <collision>
+            <origin xyz="-0.0175 -0.0025 0.0" rpy="0 0 0"/>
+            <geometry>
+                <box size="0.035 0.005 0.004"/>
+            </geometry>
+        </collision>
     </link>
     <link name="gripper_finger_right">
@@ -251,12 +247,10 @@
         </geometry>
         </visual>
-        <!--
-        <collision>
-            <origin xyz="0 0 0.025" rpy="0 0 -${PI / 2}"/>
-            <geometry>
-                <cylinder radius="0.015" length="0.05"/>
-            </geometry>
-        </collision>
-        -->
+        <collision>
+            <origin xyz="0.00525 0.026 0.00775" rpy="0 0 0"/>
+            <geometry>
+                <box size="0.0185 0.06 0.0155"/>
+            </geometry>
+        </collision>
     </link>
     <link name="gripper_finger_left">
@@ -268,12 +262,10 @@
         </geometry>
         </visual>
-        <!--
-        <collision>
-            <origin xyz="0 0 0.025" rpy="0 0 -${PI / 2}"/>
-            <geometry>
-                <cylinder radius="0.015" length="0.05"/>
-            </geometry>
-        </collision>
-        -->
+        <collision>
+            <origin xyz="0.00525 0.026 0.00775" rpy="0 0 0"/>
+            <geometry>
+                <box size="0.0185 0.06 0.0155"/>
+            </geometry>
+        </collision>
     </link>
     <!-- Joints -->

Commit message: IK point now is between the claws of the gripper

File: ws_thor/src/thor_urdf/urdf/thor.urdf.xacro (robot description, xacro)
@@ -179,4 +179,7 @@
         </collision>
     </link>
+    <link name="gripper_mid_point">
+        <xacro:default_inertial mass="1.0"/>
+    </link>
     <link name="gripper_arm_gear_right">
         <xacro:default_inertial mass="1.0"/>
@@ -328,4 +331,9 @@
         <origin xyz="0 0 0.043"/>
     </joint>
+    <joint name="gripperbase_to_midpoint" type="fixed">
+        <parent link="gripper_base"/>
+        <child link="gripper_mid_point"/>
+        <origin xyz="0 0 0.075" rpy="0 0 0"/>
+    </joint>
     <joint name="gripperbase_to_armgearright" type="revolute">
         <parent link="gripper_base"/>
